Commit message: 11

File: src/bobac3_description/xacro/basic_kit.xacro (robot description, xacro)
@@ -1,19 +1,31 @@
 <?xml version="1.0"?>
-<robot xmlns:xacro="http://www.ros.org/wiki/xacro" name="basic_kit">
-  <xacro:macro name="basic_kit" params="parent sim laser_type">
-    <joint name="extra_kit_joint" type="fixed">
+<robot xmlns:xacro="http://www.ros.org/wiki/xacro"
+       name="basic_kit">
+  <xacro:macro name="basic_kit"
+               params="parent sim laser_type">
+    <!-- ================================================== -->
+    <!-- Basic kit 与机器人主体连接 -->
+    <!-- ================================================== -->
+    <joint name="extra_kit_joint"
+           type="fixed">
       <parent link="${parent}" />
       <child link="basic_kit_link" />
       <xacro:if value="${laser_type == 'CSPC'}">
-        <origin xyz="-0.199 0 -0.02" rpy="0 0 0" />
+        <origin
+          xyz="-0.199 0 -0.02"
+          rpy="0 0 0" />
       </xacro:if>
       <xacro:unless value="${laser_type == 'CSPC'}">
-        <origin xyz="-0.034 0 0" rpy="0 0 0" />
+        <origin
+          xyz="-0.034 0 0"
+          rpy="0 0 0" />
       </xacro:unless>
       <axis xyz="0 0 0" />
     </joint>
+    <!-- ================================================== -->
+    <!-- CSPC basic kit -->
+    <!-- ================================================== -->
     <xacro:if value="${laser_type == 'CSPC'}">
-      <link
-        name="basic_kit_link">
+      <link name="basic_kit_link">
         <inertial>
           <origin
@@ -38,6 +50,5 @@
               filename="package://bobac3_description/meshes/basic_kit_link_cspc.STL" />
           </geometry>
-          <material
-            name="">
+          <material name="">
             <color
               rgba="1 1 1 1" />
@@ -55,4 +66,7 @@
       </link>
     </xacro:if>
+    <!-- ================================================== -->
+    <!-- 非 CSPC basic kit -->
+    <!-- ================================================== -->
     <xacro:unless value="${laser_type == 'CSPC'}">
       <link name="basic_kit_link">
@@ -79,6 +93,5 @@
               filename="package://bobac3_description/meshes/basic_kit_link.STL" />
           </geometry>
-          <material
-            name="">
+          <material name="">
             <color
               rgba="1 1 1 1" />
@@ -96,7 +109,9 @@
       </link>
     </xacro:unless>
+    <!-- ================================================== -->
+    <!-- Top Camera 实体模型 -->
+    <!-- ================================================== -->
     <xacro:if value="${laser_type == 'CSPC'}">
-      <link
-        name="top_camera_link">
+      <link name="top_camera_link">
         <inertial>
           <origin
@@ -121,6 +136,5 @@
               filename="package://bobac3_description/meshes/top_camera_link.STL" />
           </geometry>
-          <material
-            name="">
+          <material name="">
             <color
               rgba="1 1 1 1" />
@@ -138,4 +152,7 @@
       </link>
     </xacro:if>
+    <!-- ================================================== -->
+    <!-- 非 CSPC Top Camera -->
+    <!-- ================================================== -->
     <xacro:unless value="${laser_type == 'CSPC'}">
       <link name="top_camera_link">
@@ -162,6 +179,5 @@
               filename="package://bobac3_description/meshes/top_camera_link.STL" />
           </geometry>
-          <material
-            name="">
+          <material name="">
             <color
               rgba="0.5 0.5 0.5 1" />
@@ -179,5 +195,10 @@
       </link>
     </xacro:unless>
-    <joint name="top_camera_joint" type="fixed">
+    <!-- ================================================== -->
+    <!-- Top Camera 安装位置 -->
+    <!-- 保持官方 CSPC 安装位置 -->
+    <!-- ================================================== -->
+    <joint name="top_camera_joint"
+           type="fixed">
       <xacro:if value="${laser_type == 'CSPC'}">
         <origin
@@ -197,10 +218,33 @@
         xyz="0 0 0" />
     </joint>
+    <!-- ================================================== -->
+    <!-- 官方 v1.0.1 新增 -->
+    <!-- Top Camera optical frame -->
+    <!-- Gazebo Camera Sensor 使用这个 frame -->
+    <!-- ================================================== -->
+    <link name="top_camera_optical_link" />
+    <joint name="top_camera_optical_joint"
+           type="fixed">
+      <parent
+        link="top_camera_link" />
+      <child
+        link="top_camera_optical_link" />
+      <origin
+        xyz="0 0 0"
+        rpy="0 0.78 0" />
+    </joint>
+    <!-- ================================================== -->
+    <!-- Gazebo 外观 -->
+    <!-- ================================================== -->
     <xacro:if value="${sim}">
       <gazebo reference="basic_kit_link">
-        <material>Gazebo/White</material>
+        <material>
+          Gazebo/White
+        </material>
       </gazebo>
       <gazebo reference="top_camera_link">
-        <material>Gazebo/DarkGrey</material>
+        <material>
+          Gazebo/DarkGrey
+        </material>
       </gazebo>
     </xacro:if>

File: src/bobac3_description/xacro/bobac3_base.xacro (robot description, xacro)
@@ -518,5 +518,5 @@
     <joint name="base_berxel_camera_joint" type="fixed">
       <origin
-        xyz="0.176804013961284 0 0.7875"
+        xyz="0.176804013961284 0 0.149"
         rpy="0 0 0" />
       <parent

File: src/bobac3_description/xacro/gazebo_plugin.xacro (robot description, xacro)
@@ -1,14 +1,33 @@
 <?xml version="1.0"?>
-<robot xmlns:xacro="http://www.ros.org/wiki/xacro" name="bobac3_gazebo_plugin">
+<robot xmlns:xacro="http://www.ros.org/wiki/xacro"
+       name="bobac3_gazebo_plugin">
   <xacro:macro name="bobac3_gazebo_plugin">
+    <!-- ================================================== -->
+    <!-- Gazebo planar move -->
+    <!-- ================================================== -->
     <gazebo>
-      <plugin name="object_controller" filename="libgazebo_ros_planar_move.so">
-        <commandTopic>cmd_vel</commandTopic>
-        <odometryTopic>odom</odometryTopic>
-        <odometryFrame>odom</odometryFrame>
-        <odometryRate>10.0</odometryRate>
-        <robotBaseFrame>base_footprint</robotBaseFrame>
+      <plugin
+        name="object_controller"
+        filename="libgazebo_ros_planar_move.so">
+        <commandTopic>
+          cmd_vel
+        </commandTopic>
+        <odometryTopic>
+          odom
+        </odometryTopic>
+        <odometryFrame>
+          odom
+        </odometryFrame>
+        <odometryRate>
+          10.0
+        </odometryRate>
+        <robotBaseFrame>
+          base_footprint
+        </robotBaseFrame>
       </plugin>
     </gazebo>
+    <!-- ================================================== -->
+    <!-- Robot materials -->
+    <!-- ================================================== -->
     <gazebo reference="charge_port_link">
       <material>Gazebo/Orange</material>
@@ -47,124 +66,378 @@
       <material>Gazebo/FlatBlack</material>
     </gazebo>
+    <!-- ================================================== -->
+    <!-- Fuse lidar -->
+    <!-- ================================================== -->
     <gazebo reference="fuse_lidar_link">
-      <material>Gazebo/BlueLaser</material>
-      <sensor type="ray" name="rplidar_sensor">
-        <pose>0 0 0 0 0 0</pose>
-        <visualize>false</visualize>
-        <update_rate>10</update_rate>
+      <material>
+        Gazebo/BlueLaser
+      </material>
+      <sensor
+        type="ray"
+        name="rplidar_sensor">
+        <pose>
+          0 0 0 0 0 0
+        </pose>
+        <visualize>
+          false
+        </visualize>
+        <update_rate>
+          10
+        </update_rate>
         <ray>
           <scan>
             <horizontal>
-              <samples>720</samples>
-              <resolution>1</resolution>
-              <min_angle>-3.14159</min_angle>
-              <max_angle>3.14159</max_angle>
+              <samples>
+                720
+              </samples>
+              <resolution>
+                1
+              </resolution>
+              <min_angle>
+                -3.14159
+              </min_angle>
+              <max_angle>
+                3.14159
+              </max_angle>
             </horizontal>
           </scan>
           <range>
-            <min>0.2</min>
-            <max>30.0</max>
-            <resolution>0.01</resolution>
+            <min>
+              0.2
+            </min>
+            <max>
+              30.0
+            </max>
+            <resolution>
+              0.01
+            </resolution>
           </range>
           <noise>
-            <type>gaussian</type>
-            <!-- Noise parameters based on published spec for Hokuyo laser
-                 achieving "+-30mm" accuracy at range < 10m.  A mean of 0.0m and
-                 stddev of 0.01m will put 99.7% of samples within 0.03m of the true
-                 reading. -->
-            <mean>0.0</mean>
-            <stddev>0.01</stddev>
+            <type>
+              gaussian
+            </type>
+            <mean>
+              0.0
+            </mean>
+            <stddev>
+              0.01
+            </stddev>
           </noise>
         </ray>
-        <plugin name="bobac3_fuse_lidar" filename="libgazebo_ros_laser.so">
-          <topicName>/scan</topicName>
-          <frameName>fuse_lidar_link</frameName>
+        <plugin
+          name="bobac3_fuse_lidar"
+          filename="libgazebo_ros_laser.so">
+          <topicName>
+            /scan
+          </topicName>
+          <frameName>
+            fuse_lidar_link
+          </frameName>
         </plugin>
       </sensor>
     </gazebo>
+    <!-- ================================================== -->
+    <!-- Bottom Camera -->
+    <!-- 保持原有 AR 充电摄像头 -->
+    <!-- ================================================== -->
     <gazebo reference="bottom_camera_link">
-      <material>Gazebo/FlatBlack</material>
-      <sensor type="camera" name="bottom_camera">
-        <update_rate>30.0</update_rate>
+      <material>
+        Gazebo/FlatBlack
+      </material>
+      <sensor
+        type="camera"
+        name="bottom_camera">
+        <update_rate>
+          30.0
+        </update_rate>
         <camera name="bottom">
-          <horizontal_fov>1.3962634</horizontal_fov>
+          <horizontal_fov>
+            1.3962634
+          </horizontal_fov>
           <image>
-            <width>720</width>
-            <height>640</height>
-            <format>R8G8B8</format>
+            <width>
+              720
+            </width>
+            <height>
+              640
+            </height>
+            <format>
+              R8G8B8
+            </format>
           </image>
           <clip>
-            <near>0.02</near>
-            <far>300</far>
+            <near>
+              0.02
+            </near>
+            <far>
+              300
+            </far>
           </clip>
           <noise>
-            <type>gaussian</type>
-            <!-- Noise is sampled independently per pixel on each frame.
-                 That pixel's noise value is added to each of its color
-                 channels, which at that point lie in the range [0,1]. -->
-            <mean>0.0</mean>
-            <stddev>0.007</stddev>
+            <type>
+              gaussian
+            </type>
+            <mean>
+              0.0
+            </mean>
+            <stddev>
+              0.007
+            </stddev>
           </noise>
         </camera>
-        <plugin name="bottom_camera" filename="libgazebo_ros_camera.so">
-          <alwaysOn>true</alwaysOn>
-          <updateRate>0.0</updateRate>
-          <cameraName>/bottom_camera</cameraName>
-          <imageTopicName>image_raw</imageTopicName>
-          <cameraInfoTopicName>camera_info</cameraInfoTopicName>
-          <frameName>bottom_camera_optical_link</frameName>
-          <hackBaseline>0.07</hackBaseline>
-          <distortionK1>0.0</distortionK1>
-          <distortionK2>0.0</distortionK2>
-          <distortionK3>0.0</distortionK3>
-          <distortionT1>0.0</distortionT1>
-          <distortionT2>0.0</distortionT2>
+        <plugin
+          name="bottom_camera"
+          filename="libgazebo_ros_camera.so">
+          <alwaysOn>
+            true
+          </alwaysOn>
+          <updateRate>
+            0.0
+          </updateRate>
+          <cameraName>
+            /bottom_camera
+          </cameraName>
+          <imageTopicName>
+            image_raw
+          </imageTopicName>
+          <cameraInfoTopicName>
+            camera_info
+          </cameraInfoTopicName>
+          <frameName>
+            bottom_camera_optical_link
+          </frameName>
+          <hackBaseline>
+            0.07
+          </hackBaseline>
+          <distortionK1>
+            0.0
+          </distortionK1>
+          <distortionK2>
+            0.0
+          </distortionK2>
+          <distortionK3>
+            0.0
+          </distortionK3>
+          <distortionT1>
+            0.0
+          </distortionT1>
+          <distortionT2>
+            0.0
+          </distortionT2>
         </plugin>
       </sensor>
     </gazebo>
-    <link name="gazebo_depth_optical_link" />
-    <joint name="gazebo_depth_camera_joint" type="fixed">
-      <parent link="bobac3_base/Cam_base_link" />
-      <child link="gazebo_depth_optical_link" />
-      <origin xyz="0 0 0" rpy="-1.57079 0 -1.57079" />
+    <!-- ================================================== -->
+    <!-- 官方 v1.0.1 新增 Top Camera -->
+    <!--
+        输出：
+        /top_camera/image_raw
+        /top_camera/camera_info
+    -->
+    <!-- ================================================== -->
+    <gazebo reference="top_camera_optical_link">
+      <material>
+        Gazebo/FlatBlack
+      </material>
+      <sensor
+        type="camera"
+        name="top_camera">
+        <update_rate>
+          30.0
+        </update_rate>
+        <camera name="top">
+          <horizontal_fov>
+            1.3962634
+          </horizontal_fov>
+          <image>
+            <width>
+              720
+            </width>
+            <height>
+              640
+            </height>
+            <format>
+              R8G8B8
+            </format>
+          </image>
+          <clip>
+            <near>
+              0.02
+            </near>
+            <far>
+              300
+            </far>
+          </clip>
+          <noise>
+            <type>
+              gaussian
+            </type>
+            <mean>
+              0.0
+            </mean>
+            <stddev>
+              0.007
+            </stddev>
+          </noise>
+        </camera>
+        <plugin
+          name="top_camera"
+          filename="libgazebo_ros_camera.so">
+          <alwaysOn>
+            true
+          </alwaysOn>
+          <updateRate>
+            0.0
+          </updateRate>
+          <cameraName>
+            /top_camera
+          </cameraName>
+          <imageTopicName>
+            image_raw
+          </imageTopicName>
+          <cameraInfoTopicName>
+            camera_info
+          </cameraInfoTopicName>
+          <frameName>
+            top_camera_optical_link
+          </frameName>
+          <hackBaseline>
+            0.07
+          </hackBaseline>
+          <distortionK1>
+            0.0
+          </distortionK1>
+          <distortionK2>
+            0.0
+          </distortionK2>
+          <distortionK3>
+            0.0
+          </distortionK3>
+          <distortionT1>
+            0.0
+          </distortionT1>
+          <distortionT2>
+            0.0
+          </distortionT2>
+        </plugin>
+      </sensor>
+    </gazebo>
+    <!-- ================================================== -->
+    <!-- Berxel RGB-D Camera -->
+    <!-- 保留，但以后不再负责任务三目标识别 -->
+    <!-- ================================================== -->
+    <link
+      name="gazebo_depth_optical_link" />
+    <joint
+      name="gazebo_depth_camera_joint"
+      type="fixed">
+      <parent
+        link="bobac3_base/Cam_base_link" />
+      <child
+        link="gazebo_depth_optical_link" />
+      <origin
+        xyz="0 0 0"
+        rpy="-1.57079 0 -1.57079" />
     </joint>
     <gazebo reference="bobac3_base/Cam_base_link">
-      <sensor name="berxel_base_camera" type="depth">
-        <update_rate>20</update_rate>
+      <sensor
+        name="berxel_base_camera"
+        type="depth">
+        <update_rate>
+          20
+        </update_rate>
         <camera>
-          <horizontal_fov>1.047198</horizontal_fov>
+          <horizontal_fov>
+            1.047198
+          </horizontal_fov>
           <image>
-            <width>640</width>
-            <height>480</height>
-            <format>R8G8B8</format>
+            <width>
+              640
+            </width>
+            <height>
+              480
+            </height>
+            <format>
+              R8G8B8
+            </format>
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